Commit message: wheels tweeking

File: description/camera.xacro (robot description, xacro)
@@ -4,5 +4,5 @@
         <parent link="chassis"/>
         <child link="camera_link"/>
-        <origin xyz="0.276 0 0.181" rpy="0 0 0"/>
+        <origin xyz="0.276 0 0.14" rpy="0 0 0"/>
     </joint>
     <link name="camera_link">

File: description/ros2_control.xacro (robot description, xacro)
@@ -11,10 +11,10 @@
                 <param name="baud_rate">57600</param>
                 <param name="timeout">1000</param>
-                <param name="enc_counts_per_rev">7406</param>
+                <param name="enc_counts_per_rev">9100</param>
             </hardware>
             <joint name="left_wheel_joint">
                 <command_interface name="velocity">
-                    <param name="min">-10</param>
-                    <param name="max">10</param>
+                    <param name="min">-4</param>
+                    <param name="max">4</param>
                 </command_interface>
                 <state_interface name="velocity"/>
@@ -23,6 +23,6 @@
             <joint name="right_wheel_joint">
                 <command_interface name="velocity">
-                    <param name="min">-10</param>
-                    <param name="max">10</param>
+                    <param name="min">-4</param>
+                    <param name="max">4</param>
                 </command_interface>
                 <state_interface name="velocity"/>
